File: eagle-files/design1.sch (EAGLE design)
At the start: 42 parts, among them IC2 STM32L011F3U6TR, IC3 TPS54308DDCR, IC4 MCP6486T-E/OT, Q1 BSS138, Q2 SI3481DV, X1 DG3XX-02-5.0

Commit message: Update hardware + add state machine
Software: Add state machine
Hardware: Add EXT interrupt zener diode
Hardware: Add diode to prevent buck converter reverse current
Other:
- note added: "To create stable circuitry Additional diode in needed here 512-SS24FL 40V 2A SCHOTTKY"
Changed lines of the file:
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@@
 <text x="99.06" y="83.82" size="1.27" layer="95">Low Forward Voltage Drop Diode (approx 0.3)</text>
 <text x="147.32" y="71.12" size="1.778" layer="95">0.596 V</text>
+<text x="162.56" y="126.365" size="1.778" layer="94">To create stable circuitry
+Additional diode in needed here
+512-SS24FL 40V 2A SCHOTTKY</text>
+<wire x1="160.02" y1="134.62" x2="160.02" y2="124.46" width="0.1524" layer="95"/>
+<wire x1="160.02" y1="124.46" x2="175.26" y2="124.46" width="0.1524" layer="95"/>
+<wire x1="175.26" y1="124.46" x2="200.66" y2="124.46" width="0.1524" layer="95"/>
+<wire x1="200.66" y1="124.46" x2="200.66" y2="134.62" width="0.1524" layer="95"/>
+<wire x1="200.66" y1="134.62" x2="160.02" y2="134.62" width="0.1524" layer="95"/>
+<wire x1="175.26" y1="113.03" x2="175.26" y2="124.46" width="0.1524" layer="95"/>
+<wire x1="173.99" y1="114.3" x2="175.26" y2="113.03" width="0.1524" layer="95"/>
+<wire x1="175.26" y1="113.03" x2="176.53" y2="114.3" width="0.1524" layer="95"/>
 </plain>
 <instances>
@@
 </schematic>
 </drawing>
+<compatibility>
+<note version="6.3" minversion="6.2.2" severity="warning">
+Since Version 6.2.2 text objects can contain more than one line,
+which will not be processed correctly with this version.
+</note>
+</compatibility>
 </eagle>
