File: eagle-files/design1.sch (EAGLE design)
At the start: 42 parts, among them IC2 STM32L011F3U6TR, IC3 TPS54308DDCR, IC4 MCP6486T-E/OT, Q1 BSS138, Q2 SI3481DV, X1 DG3XX-02-5.0

Commit message: Update scheme eagle
Other:
- note added: "These pin could be used for: - informing application MCU, energy storage is charging - informing application MCU, energy storage is fully charger by small pulse"
Changed lines of the file:
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@@
 <text x="96.52" y="27.305" size="1.778" layer="94">Add boot button</text>
 <wire x1="86.36" y1="35.56" x2="93.98" y2="30.48" width="0.1524" layer="95"/>
+<wire x1="121.92" y1="48.26" x2="121.92" y2="116.84" width="0.1524" layer="95"/>
+<wire x1="121.92" y1="116.84" x2="99.06" y2="116.84" width="0.1524" layer="95"/>
+<wire x1="99.06" y1="116.84" x2="99.06" y2="127" width="0.1524" layer="95"/>
+<wire x1="99.06" y1="127" x2="187.96" y2="127" width="0.1524" layer="95"/>
+<wire x1="187.96" y1="127" x2="187.96" y2="116.84" width="0.1524" layer="95"/>
+<wire x1="187.96" y1="116.84" x2="121.92" y2="116.84" width="0.1524" layer="95"/>
+<text x="101.6" y="118.745" size="1.778" layer="94">These pin could be used for:
+- informing application MCU, energy storage is charging
+- informing application MCU, energy storage is fully charger by small pulse</text>
 </plain>
 <instances>

Commit message: Changes to PCB required
Other:
- note added: "Add digital potentiometer in series with R12 to control output voltage and reduce output power if input voltage is not sufficient enough"
Changed lines of the file:
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@@
 Zener diode MM3Z3V0T1G + 47k resistor
 Connect with PA10</text>
+<wire x1="35.56" y1="15.24" x2="22.86" y2="15.24" width="0.1524" layer="95"/>
+<wire x1="22.86" y1="15.24" x2="22.86" y2="-10.16" width="0.1524" layer="95"/>
+<wire x1="22.86" y1="-10.16" x2="30.48" y2="-10.16" width="0.1524" layer="95"/>
+<wire x1="30.48" y1="-10.16" x2="30.48" y2="-5.08" width="0.1524" layer="95"/>
+<wire x1="30.48" y1="-5.08" x2="81.28" y2="-5.08" width="0.1524" layer="95"/>
+<wire x1="81.28" y1="-5.08" x2="81.28" y2="-20.32" width="0.1524" layer="95"/>
+<wire x1="81.28" y1="-20.32" x2="30.48" y2="-20.32" width="0.1524" layer="95"/>
+<wire x1="30.48" y1="-20.32" x2="30.48" y2="-10.16" width="0.1524" layer="95"/>
+<text x="33.02" y="-17.78" size="1.778" layer="95">Add digital potentiometer in series with R12
+to control output voltage and reduce
+ output power if input voltage is not
+sufficient enough</text>
 </plain>
 <instances>
